File: Files/Board/nostrum.kicad_pcb (KiCad board)
At the start: 2 copper layers, 115 x 89.7 mm, 51 parts

Commit message: Updates
Parts:
- moved ? 2.12 mm to (84.3, 23.7)
Changed lines of the file:
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@@
   )
   (footprint "Library:MountingHole_2.2mm_M2draw" (layer "F.Cu")
-    (at 85.082288 25.672981)
+    (at 84.295081 23.703531)
     (descr "Mounting Hole 2.2mm, no annular, M2")
     (tags "mounting hole 2.2mm no annular m2")
